Commit message: add transmission attribute for T_module

File: mr_description/urdf/T_module/T_module.urdf.xacro (robot description, xacro)
@@ -72,4 +72,17 @@
     <limit  lower="-2.07" upper="2.07"  effort="0"  velocity="0" />
   </joint>
+  <!--    test reduction ratio-->
+  <transmission name="simple_trans">
+    <type>transmission_interface/SimpleTransmission</type>
+    <joint name="${name}_Joint">
+      <hardwareInterface>PositionJointInterface</hardwareInterface>
+      <hardwareInterface>VelocityJointInterface</hardwareInterface>
+    </joint>
+    <actuator name="${name}_motor">
+      <mechanicalReduction>480</mechanicalReduction>
+      <hardwareInterface>PositionJointInterface</hardwareInterface>
+      <hardwareInterface>VelocityJointInterface</hardwareInterface>
+    </actuator>
+  </transmission>
 <!--the TModule_OutLink in T module-->
   <link  name="${name}_OutLink_2">

Commit message: add candump_pdo.sh

File: mr_description/urdf/T_module/T_module.urdf.xacro (robot description, xacro)
@@ -65,10 +65,10 @@
   </link>
 <!-- joint between TModule_InLink and TModule_OutLink -->
-  <joint  name="${name}_Joint"  type="revolute">
+  <joint  name="${name}_Joint"  type="continuous">
     <origin  xyz="0 0 0.1466"  rpy="-1.5708 1.2251E-16 -3.1416" />
     <parent  link="${name}_InLink_1" />
     <child   link="${name}_OutLink_2" />
     <axis   xyz="0 0 1" />
-    <limit  lower="-2.07" upper="2.07"  effort="0"  velocity="0" />
+<!--    <limit  lower="-2.07" upper="2.07"  effort="0"  velocity="0" />-->
   </joint>
   <!--    test reduction ratio-->
@@ -91,5 +91,5 @@
       <mass  value="1.4322" />
       <inertia   ixx="0.0018144"  ixy="-1.0634E-06"  ixz="9.3521E-08"
-      					 iyy="0.0011673"  iyz="8.3209E-05"  izz="0.0023046" />
+      		iyy="0.0011673"  iyz="8.3209E-05"  izz="0.0023046" />
     </inertial>
     <visual>

File: mr_description/urdf/T_module/T_module_only.urdf.xacro (robot description, xacro)
@@ -14,11 +14,5 @@
        is the world frame). For more, see http://www.ros.org/wiki/xacro -->
   <!-- foot for module arm-->
-  <link name="base_link">
-    <inertial>
-	<origin xyz="0 0 0" rpy="0 0 0"/>
-	<mass value="1.0"/>
-	<inertia ixx="0.1"  ixy="0"  ixz="0" iyy="0.1" iyz="0" izz="0.1" />
-    </inertial>
-  </link>
+  <link name="base_link"/>
   <xacro:T_module name="T" parent="base_link">
     <origin xyz="0 0 0" rpy="0 0 0" />
