Commit message: I_module test successed

File: mr_description/urdf/I_module/I_module.urdf.xacro (robot description, xacro)
@@ -64,10 +64,10 @@
   </link>
 <!-- joint between IModule_InLink and IModule_OutLink -->
-  <joint  name="${name}_Joint"  type="revolute">
+  <joint  name="${name}_Joint"  type="continuous">
     <origin  xyz="0 0 0.12015" rpy="0 0 0" />
     <parent  link="${name}_InLink_1" />
     <child   link="${name}_OutLink_2" />
     <axis   xyz="0 0 1" />
-    <limit  lower="-3.14"  upper="3.14"  effort="0"  velocity="0" />
+<!--    <limit  lower="-3.14"  upper="3.14"  effort="0"  velocity="0" />-->
   </joint>
   <!--    test reduction ratio-->
@@ -79,5 +79,5 @@
     </joint>
     <actuator name="${name}_motor">
-      <mechanicalReduction>110</mechanicalReduction>
+      <mechanicalReduction>457</mechanicalReduction>
       <hardwareInterface>PositionJointInterface</hardwareInterface>
       <hardwareInterface>VelocityJointInterface</hardwareInterface>

File: mr_description/urdf/T_module/T_module.urdf.xacro (robot description, xacro)
@@ -65,5 +65,5 @@
   </link>
 <!-- joint between TModule_InLink and TModule_OutLink -->
-  <joint  name="${name}_Joint_2"  type="revolute">
+  <joint  name="${name}_Joint"  type="revolute">
     <origin  xyz="0 0 0.1466"  rpy="-1.5708 1.2251E-16 -3.1416" />
     <parent  link="${name}_InLink_1" />

Commit message: modify joint limits in URDF

File: mr_description/urdf/I_module/I_module.urdf.xacro (robot description, xacro)
@@ -69,5 +69,5 @@
     <child   link="${name}_OutLink_2" />
     <axis   xyz="0 0 1" />
-<!--    <limit  lower="-3.14"  upper="3.14"  effort="0"  velocity="0" />-->
+    <limit   effort="75"  velocity="1.1" />
   </joint>
   <!--    test reduction ratio-->

File: mr_description/urdf/T_module/T_module.urdf.xacro (robot description, xacro)
@@ -65,15 +65,16 @@
   </link>
 <!-- joint between TModule_InLink and TModule_OutLink -->
-  <joint  name="${name}_Joint"  type="continuous">
+  <joint  name="${name}_Joint"  type="revolute">
+<!--  <joint  name="${name}_Joint"  type="continuous">-->
     <origin  xyz="0 0 0.1466"  rpy="-1.5708 1.2251E-16 -3.1416" />
     <parent  link="${name}_InLink_1" />
     <child   link="${name}_OutLink_2" />
     <axis   xyz="0 0 1" />
-<!--    <limit  lower="-2.07" upper="2.07"  effort="0"  velocity="0" />-->
+    <limit  lower="-2.07" upper="2.07"  effort="75"  velocity="1.047" />
   </joint>
   <!--    test reduction ratio-->
-  <transmission name="simple_trans">
+  <transmission name="${name}_trans">
     <type>transmission_interface/SimpleTransmission</type>
-    <joint name="${name}_Joint">
+    <joint name="${name}_Joint" >
       <hardwareInterface>PositionJointInterface</hardwareInterface>
       <hardwareInterface>VelocityJointInterface</hardwareInterface>
