Commit message: modify manipulator urdf

File: mr_description/robots/moduleManipulator.urdf.xacro (robot description, xacro)
@@ -36,18 +36,18 @@
     <origin xyz="0 0 0" rpy="0 0 0" />
   </xacro:I_module>
-  <xacro:T_module name="T2" parent="I1_Lr_Link_3">
+  <xacro:T_invert name="T2" parent="I1_Lr_Link_3" >
+    <origin xyz="0 0 0" rpy="0 0 0" />
+  </xacro:T_invert>
+  <xacro:T_module name="T3" parent="T2_Lr_Link_0">
+    <origin xyz="0 0 0.005" rpy="0 0 ${pi}" />
+  </xacro:T_module>
+  <xacro:I_module name="I4" parent="T3_Lr_Link_3">
+    <origin xyz="0 0 0" rpy="0 0 0" />
+  </xacro:I_module>
+  <xacro:T_module name="T5" parent="I4_Lr_Link_3">
     <origin xyz="0 0 0" rpy="0 0 0" />
   </xacro:T_module>
-  <xacro:T_invert name="T3" parent="T2_Lr_Link_3" >
-    <origin xyz="0 0 0.005" rpy="0 0 0" />
-  </xacro:T_invert>
-  <xacro:T_module name="T4" parent="T3_Lr_Link_0">
-    <origin xyz="0 0 0" rpy="0 0 0" />
-  </xacro:T_module>
-  <xacro:I_module name="I5" parent="T4_Lr_Link_3">
-    <origin xyz="0 0 0" rpy="0 0 0" />
-  </xacro:I_module>
-  <xacro:G_module name="G6" parent="I5_Lr_Link_3">
-    <origin xyz="0 0 0" rpy="${pi*0.5} 0 0" />
+  <xacro:G_module name="G6" parent="T5_Lr_Link_3">
+    <origin xyz="0 0 0" rpy="${pi*0.5} 0 ${pi*0.5}" />
   </xacro:G_module>
 <!--  <xacro:I_module name="_I5" parent="base_link">-->

File: mr_description/urdf/G_module.urdf.xacro (robot description, xacro)
@@ -46,5 +46,5 @@
   </link>
 <!--  joint between the palm and the left finger-->
-  <joint name="${name}_finger_joint_l"
+  <joint name="${name}_Joint"
     type="prismatic">
     <origin
@@ -58,9 +58,22 @@
       upper="0.04"
       effort="0"
-      velocity="0" />
+      velocity="0.1" />
     <dynamics
       damping="1"
       friction="1" />
   </joint>
+   <!-- test reduction ratio-->
+  <transmission name="simple_trans">
+    <type>transmission_interface/SimpleTransmission</type>
+    <joint name="${name}_Joint">
+      <hardwareInterface>PositionJointInterface</hardwareInterface>
+      <hardwareInterface>VelocityJointInterface</hardwareInterface>
+    </joint>
+    <actuator name="${name}_motor">
+      <mechanicalReduction>400</mechanicalReduction>
+      <hardwareInterface>PositionJointInterface</hardwareInterface>
+      <hardwareInterface>VelocityJointInterface</hardwareInterface>
+    </actuator>
+  </transmission>
 <!--  the left finger link-->
   <link name="${name}_finger_link_l">
@@ -108,5 +121,5 @@
       upper="0.04"
       effort="0"
-      velocity="0" />
+      velocity="0.1" />
     <dynamics
       damping="1"

File: mr_description/urdf/I_module/I_module.urdf.xacro (robot description, xacro)
@@ -107,5 +107,5 @@
   </link>
 <!-- joint between IModule_OutLink and Lockring_Link -->
-		<joint name="${name}_Lr_Joint_3" type="fixed">
+    <joint name="${name}_Lr_Joint_3" type="fixed">
       <origin xyz="0 0 0.0432" rpy="0 0 0" />
       <parent link="${name}_OutLink_2" />

File: mr_description/urdf/T_module/T_Invert.urdf.xacro (robot description, xacro)
@@ -66,5 +66,5 @@
   </link>
 <!-- joint between TModule_InLink and TModule_OutLink -->
-  <joint  name="${name}_Joint_2"  type="revolute">
+  <joint  name="${name}_Joint"  type="revolute">
    <origin  xyz=" 0 0 0"  rpy="4.7124 -1.2251E-16 3.1416" />
 <!--    <origin  xyz=" 0 0 -0.1466"  rpy="4.7124 -1.2251E-16 3.1416" />-->
@@ -72,6 +72,21 @@
     <parent link="${name}_OutLink_2" />
     <axis   xyz="0 1 0" />
-    <limit  lower="-2.07" upper="2.07"  effort="0"  velocity="0" />
+    <limit  lower="-2.07" upper="2.07"  effort="75"  velocity="1.047" />
   </joint>
+  <!--    test reduction ratio-->
+  <transmission name="${name}_trans">
+    <type>transmission_interface/SimpleTransmission</type>
+    <joint name="${name}_Joint" >
+      <hardwareInterface>PositionJointInterface</hardwareInterface>
+      <hardwareInterface>VelocityJointInterface</hardwareInterface>
+<!--      <hardwareInterface>EffortJointInterface</hardwareInterface>-->
+    </joint>
+    <actuator name="${name}_motor">
+      <mechanicalReduction>480</mechanicalReduction>
+      <hardwareInterface>PositionJointInterface</hardwareInterface>
+      <hardwareInterface>VelocityJointInterface</hardwareInterface>
+<!--      <hardwareInterface>EffortJointInterface</hardwareInterface>-->
+    </actuator>
+  </transmission>
 <!--the TModule_InLink in T module-->
   <link name="${name}_InLink_1">

Commit message: add i85, t85 and g85 urdf

File: mr_description/robots/moduleManipulator.urdf.xacro (robot description, xacro)
@@ -14,4 +14,12 @@
   <!-- Gripper100 invert Module -->
   <xacro:include filename="$(find mr_description)/urdf/G_invert.urdf.xacro" />
+  <!-- 100_85_connect_link Module -->
+  <xacro:include filename="$(find mr_description)/urdf/100_85connect_link.urdf.xacro" />
+  <!-- t85 Module -->
+  <xacro:include filename="$(find mr_description)/urdf/t_module.urdf.xacro" />
+  <!-- i85  Module -->
+  <xacro:include filename="$(find mr_description)/urdf/i_module.urdf.xacro" />
+   <!-- g85  Module -->
+  <xacro:include filename="$(find mr_description)/urdf/g_module.urdf.xacro" />
 <!-- Now we can start using the macros included above to define the actual youbot -->
   <!-- The first use of a macro.  This one was defined in base.urdf.xacro above.
@@ -23,11 +31,5 @@
        is the world frame). For more, see http://www.ros.org/wiki/xacro -->
   <!-- foot for module arm-->
-  <link name="base_link">
-<!--    <inertial>    -->
-<!--	<origin xyz="0 0 0" rpy="0 0 0"/>-->
-<!--	<mass value="1.0"/>-->
-<!--	<inertia ixx="0.1"  ixy="0"  ixz="0" iyy="0.1" iyz="0" izz="0.1" />-->
-<!--    </inertial>-->
-  </link>
+  <link name="base_link"/>
 <!--  <xacro:G_invert name="G0" parent="base_link">-->
 <!--    <origin xyz="0 0 0.17836" rpy="${-pi*0.5} 0 0" />-->
@@ -42,13 +44,25 @@
     <origin xyz="0 0 0.005" rpy="0 0 ${pi}" />
   </xacro:T_module>
-  <xacro:I_module name="I4" parent="T3_Lr_Link_3">
+  <xacro:connect_link_100_85  name="cl" parent="T3_Lr_Link_3">
     <origin xyz="0 0 0" rpy="0 0 0" />
-  </xacro:I_module>
-  <xacro:T_module name="T5" parent="I4_Lr_Link_3">
+  </xacro:connect_link_100_85>
+  <xacro:i_module name="i4" parent="cl_100_85_connect_link2">
     <origin xyz="0 0 0" rpy="0 0 0" />
-  </xacro:T_module>
-  <xacro:G_module name="G6" parent="T5_Lr_Link_3">
-    <origin xyz="0 0 0" rpy="${pi*0.5} 0 ${pi*0.5}" />
-  </xacro:G_module>
+  </xacro:i_module>
+  <xacro:t_module name="t5" parent="i4_link2">
+    <origin xyz="0 0 0" rpy="0 0 ${-pi*0.5}" />
+  </xacro:t_module>
+  <xacro:g_module name="g6" parent="t5_link2">
+    <origin xyz="0 0 0.0825" rpy="0 0 0" />
+  </xacro:g_module>
+  <joint name="tcp_fixed_joint" type="fixed" >
+    <origin xyz="0 0 0.16" rpy="0 0 0" />
+    <parent link="g6_palm_link" />
+    <child link="tcp" />
+  </joint>
+  <link name="tcp"/>
+<!--  <xacro:G_module name="G6" parent="T5_Lr_Link_3">-->
+<!--    <origin xyz="0 0 0" rpy="${pi*0.5} 0 ${pi*0.5}" />-->
+<!--  </xacro:G_module>-->
 <!--  <xacro:I_module name="_I5" parent="base_link">-->
 <!--    <origin xyz="0.2 0 0" rpy="0 0 0" />-->

File: mr_description/urdf/Connect_Link.urdf.xacro (robot description, xacro)
@@ -1,4 +1,4 @@
 <?xml version="1.0"?>
-<robot xmlns:xacro="http://www.ros.org/wiki/xacro" name="ModuleManipulator">
+<robot xmlns:xacro="http://www.ros.org/wiki/xacro">
   <xacro:property name="pi" value="3.1415926535897931" />
   <xacro:property name="material_density" value="2700" />

File: mr_description/urdf/I_module/I_module.urdf.xacro (robot description, xacro)
@@ -4,9 +4,9 @@
 <xacro:macro name="I_module" params="parent name *origin">
 <!-- joint between base_link and Lockring_Link -->
-		<joint name="${name}_joint_0" type="fixed" >
-			<insert_block name="origin" />
-			<parent link="${parent}" />
-			<child link="${name}_Lr_Link_0" />
-		</joint>
+	<joint name="${name}_joint_0" type="fixed" >
+		<insert_block name="origin" />
+		<parent link="${parent}" />
+		<child link="${name}_Lr_Link_0" />
+	</joint>
 <!--the Lockring_Link in I module-->
   <link name="${name}_Lr_Link_0">
