Commit message: create moveit_config package for moduleManipulator

File: mr_description/robots/moduleManipulator.urdf (robot description, URDF)
Before this commit: robot ModuleManipulator, 25 links, 24 joints
Links:
- removed link G6_finger_link_l
- removed link G6_finger_link_r
- removed link G6_palm_link
- removed link G6_tcp
- removed link I5_InLink_1
- removed link I5_Lr_Link_0
- removed link I5_Lr_Link_3
- removed link I5_OutLink_2
- removed link T4_InLink_1
- removed link T4_Lr_Link_0
- removed link T4_Lr_Link_3
- removed link T4_OutLink_2
- added link cl_100_85_connect_link, mass 0.0438125444482135; collision cylinder length=0.022 radius=0.0425; visual mesh filename=package://mr_description/meshes/100-85_connect_link.STL
- added link cl_100_85_connect_link2
- added link g6_finger_link, mass 0.0587979869361216; collision mesh filename=package://mr_description/meshes/g_finger_link.STL; visual mesh filename=package://mr_description/meshes/g_finger_link.STL
- added link g6_finger_link1, mass 0.0587979869361215; collision mesh filename=package://mr_description/meshes/g_finger_link1.STL; visual mesh filename=package://mr_description/meshes/g_finger_link1.STL
- added link g6_palm_link, mass 0.566653469628951; collision cylinder length=0.056 radius=0.0425; visual mesh filename=package://mr_description/meshes/g_palm_link.STL
- added link i4_link, mass 0.389080654611604; collision cylinder length=0.144 radius=0.0425; visual mesh filename=package://mr_description/meshes/i_link.STL
- added link i4_link2, mass 0.80864; visual mesh filename=package://mr_description/meshes/i_link2.STL
- added link t5_link, mass 0.832217409872162; collision cylinder length=0.052 radius=0.0425; visual mesh filename=package://mr_description/meshes/t_link.STL
- added link t5_link2, mass 0.98367; collision cylinder length=0.125 radius=0.0425; visual mesh filename=package://mr_description/meshes/t_link2.STL
- added link tcp
Joints:
- removed joint G6_finger_joint_l
- removed joint G6_finger_joint_r
- removed joint G6_joint_0
- removed joint G6_tcp_joint
- removed joint I1_Joint_2
- removed joint I5_Joint_2
- removed joint I5_Lr_Joint_1
- removed joint I5_Lr_Joint_3
- removed joint I5_joint_0
- removed joint T2_Joint_2
- removed joint T3_Joint_2
- removed joint T4_Joint_2
- removed joint T4_Lr_Joint_1
- removed joint T4_Lr_Joint_3
- removed joint T4_joint_0
- added joint I1_Joint: type continuous, parent I1_InLink_1, child I1_OutLink_2, origin xyz=0 0 0.12015 rpy=0 0 0, axis 0 0 1, limit effort=75 velocity=1.1
- added joint T2_Joint: type revolute, parent T2_OutLink_2, child T2_InLink_1, origin xyz= 0 0 0 rpy=4.7124 -1.2251E-16 3.1416, axis 0 -1 0, limit lower=-2.07 upper=2.07 effort=75 velocity=1.047
- added joint T3_Joint: type revolute, parent T3_InLink_1, child T3_OutLink_2, origin xyz=0 0 0.1466 rpy=-1.5708 1.2251E-16 -3.1416, axis 0 0 -1, limit lower=-2.07 upper=2.07 effort=75 velocity=1.047
- added joint cl_fixed: type fixed, parent cl_100_85_connect_link, child cl_100_85_connect_link2, origin xyz=0 0 0.0236 rpy=0 0 0, axis 0 0 0
- added joint cl_joint_0: type fixed, parent T3_Lr_Link_3, child cl_100_85_connect_link, origin xyz=0 0 0 rpy=0 0 0
- added joint g6_Joint: type prismatic, parent g6_palm_link, child g6_finger_link, origin xyz=0 0 0 rpy=0 0 0, axis -1 0 0, limit lower=0 upper=0.06 effort=1 velocity=0.06
- added joint g6_Joint1: type prismatic, parent g6_palm_link, child g6_finger_link1, origin xyz=0 0 0 rpy=0 0 0, axis 1 0 0, limit lower=0 upper=0.06 effort=1 velocity=0.06
- added joint g6_joint_0: type fixed, parent t5_link2, child g6_palm_link, origin xyz=0 0 0.0825 rpy=0 0 0
- added joint i4_Joint: type continuous, parent i4_link, child i4_link2, origin xyz=0 0 0.137 rpy=-8.5591E-29 0 0, axis 0 0 1, limit lower=-3.1416 upper=3.1416 effort=30 velocity=1.29
- added joint i4_joint_0: type fixed, parent cl_100_85_connect_link2, child i4_link, origin xyz=0 0 0 rpy=0 0 0
- added joint t5_Joint: type revolute, parent t5_link, child t5_link2, origin xyz=0 0 0.131 rpy=0 0 3.1416, axis 1 0 0, limit lower=-2.09 upper=2.09 effort=28 velocity=2.09
- added joint t5_joint_0: type fixed, parent i4_link2, child t5_link, origin xyz=0 0 0 rpy=0 0 -1.57079632679
- added joint tcp_fixed_joint: type fixed, parent g6_palm_link, child tcp, origin xyz=0 0 0.16 rpy=0 0 0
- joint T2_Lr_Joint_1: child T2_InLink_1 -> T2_Lr_Link_0; origin xyz=0 0 0 rpy=0 0 0 -> xyz=0 0 -0.1416 rpy=0 3.1416 0; parent T2_Lr_Link_0 -> T2_InLink_1
- joint T2_Lr_Joint_3: child T2_Lr_Link_3 -> T2_OutLink_2; origin xyz=0 -0.0934 0 rpy=-1.5708 0 3.1416 -> xyz=0 0 0.0884 rpy=-1.57079632679 3.1416 3.1416; parent T2_OutLink_2 -> T2_Lr_Link_3
- joint T2_joint_0: child T2_Lr_Link_0 -> T2_Lr_Link_3
- joint T3_Lr_Joint_1: child T3_Lr_Link_0 -> T3_InLink_1; origin xyz=0 0 -0.1416 rpy=0 3.1416 0 -> xyz=0 0 0 rpy=0 0 0; parent T3_InLink_1 -> T3_Lr_Link_0
- joint T3_Lr_Joint_3: child T3_OutLink_2 -> T3_Lr_Link_3; origin xyz=0 0 0.0884 rpy=-1.57079632679 3.1416 3.1416 -> xyz=0 -0.0934 0 rpy=-1.5708 0 3.1416; parent T3_Lr_Link_3 -> T3_OutLink_2
- joint T3_joint_0: child T3_Lr_Link_3 -> T3_Lr_Link_0; origin xyz=0 0 0.005 rpy=0 0 0 -> xyz=0 0 0.005 rpy=0 0 3.14159265359; parent T2_Lr_Link_3 -> T2_Lr_Link_0

File: mr_description/urdf/g_module.urdf.xacro (robot description, xacro)
@@ -68,7 +68,7 @@
     <axis   xyz="-1 0 0" />
     <limit    lower="0"  upper="0.06" effort="1" velocity="0.06" />
-    <calibration   rising="1"   falling="1" />
-    <dynamics    damping="1"    friction="1" />
-    <safety_controller soft_upper="0.06" soft_lower="0" k_position="1" k_velocity="1" />
+<!--    <calibration   rising="1"   falling="1" />-->
+<!--    <dynamics    damping="1"    friction="1" />-->
+<!--    <safety_controller soft_upper="0.06" soft_lower="0" k_position="1" k_velocity="1" />-->
   </joint>
   <link  name="${name}_finger_link1">
@@ -106,7 +106,7 @@
     <axis   xyz="1 0 0" />
     <limit  lower="0"  upper="0.06" effort="1" velocity="0.06" />
-    <calibration  rising="1" />
-    <dynamics  damping="1"  friction="1" />
-    <safety_controller soft_upper="0.06" soft_lower="0" k_position="1" k_velocity="1" />
+<!--    <calibration  rising="1" />-->
+<!--    <dynamics  damping="1"  friction="1" />-->
+<!--    <safety_controller soft_upper="0.06" soft_lower="0" k_position="1" k_velocity="1" />-->
   </joint>
   </xacro:macro>
