Commit message: add wheeled5d robot xacro

File: mr_description/robots/manipulator6d.urdf.xacro (robot description, xacro)
@@ -1,4 +1,4 @@
 <?xml version="1.0"?>
-<robot xmlns:xacro="http://www.ros.org/wiki/xacro" name="manipulator5d">
+<robot xmlns:xacro="http://www.ros.org/wiki/xacro" name="ModuleManipulator">
   <xacro:property name="pi" value="3.1415926535897931" />
 <!-- materials for visualization -->
@@ -41,22 +41,25 @@
     <origin xyz="0 0 0" rpy="0 0 0" />
   </xacro:T_invert>
-  <xacro:T_module name="T3" parent="T2_Lr_Link_0">
-    <origin xyz="0 0 0.005" rpy="0 0 ${pi}" />
+  <xacro:I_module name="I3" parent="T2_Lr_Link_0">
+    <origin xyz="0 0 0.005" rpy="0 0 0" />
+  </xacro:I_module>
+  <xacro:T_module name="T4" parent="I3_Lr_Link_3">
+    <origin xyz="0 0 0" rpy="0 0 ${pi}" />
   </xacro:T_module>
-  <xacro:connect_link_100_85  name="cl" parent="T3_Lr_Link_3">
+  <xacro:connect_link_100_85  name="cl" parent="T4_Lr_Link_3">
     <origin xyz="0 0 0" rpy="0 0 0" />
   </xacro:connect_link_100_85>
-  <xacro:i_module name="i4" parent="cl_100_85_connect_link2">
+  <xacro:i_module name="i5" parent="cl_100_85_connect_link2">
     <origin xyz="0 0 0" rpy="0 0 0" />
   </xacro:i_module>
-  <xacro:t_module name="t5" parent="i4_link2">
+  <xacro:t_module name="t6" parent="i5_link2">
     <origin xyz="0 0 0" rpy="0 0 ${-pi*0.5}" />
   </xacro:t_module>
-  <xacro:g_module name="g6" parent="t5_link2">
+  <xacro:g_module name="g7" parent="t6_link2">
     <origin xyz="0 0 0.0825" rpy="0 0 0" />
   </xacro:g_module>
   <joint name="tcp_fixed_joint" type="fixed" >
     <origin xyz="0 0 0.16" rpy="0 0 0" />
-    <parent link="g6_palm_link" />
+    <parent link="g7_palm_link" />
     <child link="tcp" />
   </joint>

File: mr_description/robots/wheeled5d.urdf.xacro (robot description, xacro)
@@ -1,4 +1,4 @@
 <?xml version="1.0"?>
-<robot xmlns:xacro="http://www.ros.org/wiki/xacro" name="climbot5d">
+<robot xmlns:xacro="http://www.ros.org/wiki/xacro" name="wheeled5d">
   <xacro:property name="pi" value="3.1415926535897931" />
 <!-- materials for visualization -->
@@ -22,11 +22,29 @@
        the origin block defines where the component is w.r.t its parent (in this case the parent
        is the world frame). For more, see http://www.ros.org/wiki/xacro -->
-<!--    climbot move group 1-->
-  <link name="base_gripper1" />
-  <xacro:G_invert name="G0" parent="base_gripper1">
-    <origin xyz="0 0 0.17836" rpy="${-pi*0.5} 0 0" />
-  </xacro:G_invert>
-  <xacro:I_module name="I1" parent="G0_palm_link">
-    <origin xyz="0 0 0" rpy="${pi*0.5} 0 0" />
+  <link name="world" />
+  <joint name="wheel_Joint1" type="fixed">
+    <origin xyz="0 0 0.15" rpy="0 ${pi*0.5} 0"/>
+    <parent link="world"/>
+    <child link="wheel1"/>
+  </joint>
+  <link name="wheel1" >
+    <visual>
+      <origin xyz=" 0 0 -0.025" rpy="0 0 0" />
+      <geometry>
+      	<cylinder radius="0.15" length="0.05"/>
+      </geometry>
+      <material name="">
+        <color rgba="0.02 0.02 0.02 1" />
+      </material>
+    </visual>
+    <collision>
+      <origin xyz=" 0 0 -0.025" rpy="0 0 0" />
+      <geometry>
+      	<cylinder radius="0.15" length="0.05"/>
+      </geometry>
+    </collision>
+  </link>
+  <xacro:I_module name="I1" parent="wheel1">
+    <origin xyz="0 0 0" rpy="0 0 ${pi*0.5}" />
   </xacro:I_module>
   <xacro:T_module name="T2" parent="I1_Lr_Link_3">
@@ -42,32 +60,25 @@
     <origin xyz="0 0 0" rpy="0 0 0" />
   </xacro:I_module>
-  <xacro:G_module name="G6" parent="I5_Lr_Link_3">
-    <origin xyz="0 0 0" rpy="${pi*0.5} 0 0" />
-  </xacro:G_module>
-<!--    climbot move group 2-->
-<!--   <link name="base_gripper2" />-->
-<!--   -->
-<!--  <xacro:G_invert name="_G6" parent="base_gripper2">-->
-<!--    <origin xyz="0.2 0 0.17836" rpy="${-pi*0.5} 0 0" />-->
-<!--  </xacro:G_invert>-->
-<!--  <xacro:I_module name="_I5" parent="_G6_palm_link">-->
-<!--    <origin xyz="0 0 0" rpy="${pi*0.5} 0 0" />-->
-<!--  </xacro:I_module>-->
-<!--  <xacro:T_invert name="_T4" parent="_I5_Lr_Link_3">-->
-<!--    <origin xyz="0 0 0.005" rpy="0 0 0" />-->
-<!--  </xacro:T_invert>-->
-<!--  -->
-<!--  <xacro:T_module name="_T3" parent="_T4_Lr_Link_0">-->
-<!--    <origin xyz="0 0 0" rpy="0 0 0" />-->
-<!--  </xacro:T_module>-->
-<!--  <xacro:T_invert name="_T2" parent="_T3_Lr_Link_3">-->
-<!--    <origin xyz="0 0 0.005" rpy="0 0 0" />-->
-<!--  </xacro:T_invert>-->
-<!--  <xacro:I_module name="_I1" parent="_T2_Lr_Link_0">-->
-<!--    <origin xyz="0 0 0" rpy="0 0 0" />-->
-<!--  </xacro:I_module>-->
-<!--  -->
-<!--  <xacro:G_module name="_G0" parent="_I1_Lr_Link_3">-->
-<!--    <origin xyz="0 0 0" rpy="${pi*0.5} 0 0" />-->
-<!--  </xacro:G_module>-->
+  <joint name="wheel_Joint2" type="fixed">
+    <origin xyz="0 0 0.05" rpy="0 0 0"/>
+    <parent link="I5_Lr_Link_3"/>
+    <child link="wheel2"/>
+  </joint>
+  <link name="wheel2" >
+    <visual>
+      <origin xyz=" 0 0 -0.025" rpy="0 0 0" />
+      <geometry>
+      	<cylinder radius="0.15" length="0.05"/>
+      </geometry>
+      <material name="">
+        <color rgba="0.02 0.02 0.02 1" />
+      </material>
+    </visual>
+    <collision>
+      <origin xyz=" 0 0 -0.025" rpy="0 0 0" />
+      <geometry>
+      	<cylinder radius="0.15" length="0.05"/>
+      </geometry>
+    </collision>
+  </link>
 </robot>

File: mr_description/urdf/G_invert.urdf.xacro (robot description, xacro)
@@ -48,31 +48,32 @@
   </link>
 <!--  joint between the palm and the left finger-->
-  <joint name="${name}_finger_joint_l"
+  <joint name="${name}_Joint"
     type="prismatic">
-    <origin
-      xyz="0.038 0 0"
-      rpy="0 0 0" />
+    <origin xyz="0.038 0 0"  rpy="0 0 0" />
     <parent link="${name}_palm_link" />
     <child  link="${name}_finger_link_l" />
     <axis   xyz="-1 0 0" />
-    <limit
-      lower="0"
-      upper="0.04"
-      effort="0"
-      velocity="0" />
-    <dynamics
-      damping="1"
-      friction="1" />
+    <limit lower="0" upper="0.04" effort="10" velocity="0.02" />
+    <dynamics  damping="1" friction="1" />
   </joint>
+   <!-- test reduction ratio-->
+  <transmission name="simple_trans">
+    <type>transmission_interface/SimpleTransmission</type>
+    <joint name="${name}_Joint">
+      <hardwareInterface>PositionJointInterface</hardwareInterface>
+      <hardwareInterface>VelocityJointInterface</hardwareInterface>
+    </joint>
+    <actuator name="${name}_motor">
+      <mechanicalReduction>400</mechanicalReduction>
+      <hardwareInterface>PositionJointInterface</hardwareInterface>
+      <hardwareInterface>VelocityJointInterface</hardwareInterface>
+    </actuator>
+  </transmission>
 <!--  the left finger link-->
   <link name="${name}_finger_link_l">
     <inertial>
-      <origin
-        xyz="-0.053748 0.15337 2.2717E-07"
-        rpy="0 0 0" />
-      <mass
-        value="0.89853" />
-      <inertia
-        ixx="0.0023606"
+      <origin xyz="-0.053748 0.15337 2.2717E-07"  rpy="0 0 0" />
+      <mass value="0.89853" />
+      <inertia ixx="0.0023606"
         ixy="-0.00017835"
         ixz="4.9579E-09"
@@ -82,15 +83,10 @@
     </inertial>
     <visual>
-      <origin
-        xyz="0 0 0"
-        rpy="0 0 0" />
+      <origin  xyz="0 0 0"  rpy="0 0 0" />
       <geometry>
-        <mesh
-          filename="package://mr_description/meshes/finger_link_l.STL" />
+        <mesh  filename="package://mr_description/meshes/finger_link_l.STL" />
       </geometry>
-      <material
-        name="">
-        <color
-          rgba="0.52941 0.54902 0.54902 1" />
+      <material  name="">
+        <color  rgba="0.52941 0.54902 0.54902 1" />
       </material>
     </visual>
@@ -105,28 +101,17 @@
   </link>
 <!--  joint between the right finger and the palm-->
-  <joint  name="${name}_finger_joint_r" type="prismatic">
-    <origin
-      xyz="-0.038 0 0"
-      rpy="0 0 0" />
+  <joint  name="${name}_Joint1" type="prismatic">
+    <origin xyz="-0.038 0 0"  rpy="0 0 0" />
     <parent link="${name}_palm_link" />
     <child  link="${name}_finger_link_r" />
     <axis  xyz="1 0 0" />
-    <limit
-      lower="0"
-      upper="0.04"
-      effort="0"
-      velocity="0" />
-    <dynamics
-      damping="1"
-      friction="1" />
+    <limit  lower="0" upper="0.04"  effort="10" velocity="0.02" />
+    <dynamics  damping="1" friction="1" />
   </joint>
 <!-- the right finger link-->
   <link name="${name}_finger_link_r">
     <inertial>
-      <origin
-        xyz="0.053748 0.15337 -2.2717E-07"
-        rpy="0 0 0" />
-      <mass
-        value="0.89853" />
+      <origin    xyz="0.053748 0.15337 -2.2717E-07"   rpy="0 0 0" />
+      <mass  value="0.89853" />
       <inertia
         ixx="0.0023606"

File: mr_description/urdf/G_module.urdf.xacro (robot description, xacro)
@@ -29,6 +29,5 @@
         rpy="0 0 0" />
       <geometry>
-        <mesh
-          filename="package://mr_description/meshes/palm_link.STL" />
+        <mesh filename="package://mr_description/meshes/palm_link.STL" />
       </geometry>
       <material  name="">
@@ -46,20 +45,11 @@
   </link>
 <!--  joint between the palm and the left finger-->
-  <joint name="${name}_Joint"
-    type="prismatic">
-    <origin
-      xyz="0.038 0 0"
-      rpy="0 0 0" />
+  <joint name="${name}_Joint"  type="prismatic">
+    <origin xyz="0.038 0 0"  rpy="0 0 0" />
     <parent link="${name}_palm_link" />
     <child  link="${name}_finger_link_l" />
     <axis   xyz="-1 0 0" />
-    <limit
-      lower="0"
-      upper="0.04"
-      effort="0"
-      velocity="0.1" />
-    <dynamics
-      damping="1"
-      friction="1" />
+    <limit  lower="0"  upper="0.04" effort="10" velocity="0.02" />
+    <dynamics  damping="1" friction="1" />
   </joint>
    <!-- test reduction ratio-->
@@ -79,9 +69,6 @@
   <link name="${name}_finger_link_l">
     <inertial>
-      <origin
-        xyz="-0.053748 0.15337 2.2717E-07"
-        rpy="0 0 0" />
-      <mass
-        value="0.89853" />
+      <origin  xyz="-0.053748 0.15337 2.2717E-07"  rpy="0 0 0" />
+      <mass   value="0.89853" />
       <inertia
         ixx="0.0023606"
@@ -102,36 +89,26 @@
     </visual>
     <collision>
-      <origin xyz="-0.05 0.18 0" rpy="0 0 0" />
-<!--      <origin xyz="0 0 0" rpy="0 0 0" />-->
+<!--      <origin xyz="-0.05 0.18 0" rpy="0 0 0" />-->
+      <origin xyz="0 0 0" rpy="0 0 0" />
       <geometry>
-      	<box size="0.01 0.1 0.1"/>
-<!--        <mesh filename="package://mr_description/meshes/finger_link_l.STL" />-->
+<!--      	<box size="0.01 0.1 0.1"/>-->
+        <mesh filename="package://mr_description/meshes/finger_link_l.STL" />
       </geometry>
     </collision>
   </link>
 <!--  joint between the right finger and the palm-->
-  <joint  name="${name}_finger_joint_r"
-    type="prismatic">
+  <joint  name="${name}_Joint1"  type="prismatic">
     <origin  xyz="-0.038 0 0" rpy="0 0 0" />
     <parent link="${name}_palm_link" />
     <child  link="${name}_finger_link_r" />
     <axis  xyz="1 0 0" />
-    <limit
-      lower="0"
-      upper="0.04"
-      effort="0"
-      velocity="0.1" />
-    <dynamics
-      damping="1"
-      friction="1" />
+    <limit lower="0"  upper="0.04" effort="10" velocity="0.02" />
+    <dynamics   damping="1" friction="1" />
   </joint>
 <!-- the right finger link-->
   <link name="${name}_finger_link_r">
     <inertial>
-      <origin
-        xyz="0.053748 0.15337 -2.2717E-07"
-        rpy="0 0 0" />
-      <mass
-        value="0.89853" />
+      <origin   xyz="0.053748 0.15337 -2.2717E-07"  rpy="0 0 0" />
+      <mass    value="0.89853" />
       <inertia
         ixx="0.0023606"
@@ -152,9 +129,9 @@
     </visual>
     <collision>
-      <origin xyz="0.05 0.18 0" rpy="0 0 0" />
-<!--      <origin xyz="0 0 0" rpy="0 0 0" />-->
+<!--      <origin xyz="0.05 0.18 0" rpy="0 0 0" />-->
+      <origin xyz="0 0 0" rpy="0 0 0" />
       <geometry>
-      	<box size="0.01 0.1 0.1"/>
-<!--        <mesh filename="package://mr_description/meshes/finger_link_r.STL" />-->
+<!--      	<box size="0.01 0.1 0.1"/>-->
+        <mesh filename="package://mr_description/meshes/finger_link_r.STL" />
       </geometry>
     </collision>
