Commit message: mr_setup_detect now detects connection_angle between adjecent modules

File: mr_description/robots/mr_xacro_template.urdf.xacro (robot description, xacro)
@@ -30,4 +30,2 @@
        the origin block defines where the component is w.r.t its parent (in this case the parent
        is the world frame). For more, see http://www.ros.org/wiki/xacro -->
-  <!-- foot for robot-->
-  <link name="base_link"/>
