Commit message: add I_invert.urdf.xacro
change climbot5d.urdf.xacro

add I_invert.urdf.xacro and change climbot5d.urdf.xacro

modify climbot5d_invert.urdf.xacro

File: mr_description/robots/climbot5d.urdf.xacro (robot description, xacro)
@@ -8,4 +8,6 @@
   <!-- T Module -->
   <xacro:include filename="$(find mr_description)/urdf/T_module/T_module.urdf.xacro" />
+  <!-- I Invert Module -->
+  <xacro:include filename="$(find mr_description)/urdf/I_module/I_invert.urdf.xacro" />
   <!-- T Invert Module -->
   <xacro:include filename="$(find mr_description)/urdf/T_module/T_Invert.urdf.xacro" />
@@ -14,4 +16,6 @@
   <!-- Gripper100 invert Module -->
   <xacro:include filename="$(find mr_description)/urdf/G_invert.urdf.xacro" />
+  <!-- sleeve_link Module -->
+  <xacro:include filename="$(find mr_description)/urdf/sleeve_link.urdf.xacro" />
 <!-- Now we can start using the macros included above to define the actual robot -->
   <!-- The first use of a macro.  This one was defined in base.urdf.xacro above.
@@ -28,20 +32,23 @@
   </xacro:G_invert>
   <xacro:I_module name="I1" parent="G0_palm_link">
-    <origin xyz="0 0 0" rpy="${pi*0.5} 0 0" />
+    <origin xyz="0 0 0" rpy="${pi*0.5} ${-pi*0.5} 0" />
   </xacro:I_module>
-  <xacro:T_module name="T2" parent="I1_Lr_Link_3">
-    <origin xyz="0 0 0" rpy="0 0 0" />
-  </xacro:T_module>
-  <xacro:T_invert name="T3" parent="T2_Lr_Link_3" >
+  <xacro:T_invert name="T2" parent="I1_Lr_Link_3">
     <origin xyz="0 0 0.005" rpy="0 0 0" />
   </xacro:T_invert>
-  <xacro:T_module name="T4" parent="T3_Lr_Link_0">
+  <xacro:T_module name="T3" parent="T2_Lr_Link_0" >
+    <origin xyz="0 0 0.005" rpy="0 0 ${pi}" />
+  </xacro:T_module>
+  <xacro:sleeve_link name="sleeve_link" parent="T3_Lr_Link_3" >
     <origin xyz="0 0 0" rpy="0 0 0" />
+  </xacro:sleeve_link>
+  <xacro:T_module name="T4" parent="sleeve_link_link">
+    <origin xyz="0 0 ${sleeve_link_length}" rpy="0 0 0" />
   </xacro:T_module>
-  <xacro:I_module name="I5" parent="T4_Lr_Link_3">
+  <xacro:I_invert name="I5" parent="T4_Lr_Link_3">
     <origin xyz="0 0 0" rpy="0 0 0" />
-  </xacro:I_module>
+  </xacro:I_invert>
   <xacro:G_module name="G6" parent="I5_Lr_Link_3">
-    <origin xyz="0 0 0" rpy="${pi*0.5} 0 0" />
+    <origin xyz="0 0 0" rpy="${pi*0.5} 0 ${-pi*0.5}" />
   </xacro:G_module>
 <!--    climbot move group 2-->

File: mr_description/robots/climbot5d_invert.urdf.xacro (robot description, xacro)
@@ -8,4 +8,6 @@
   <!-- T Module -->
   <xacro:include filename="$(find mr_description)/urdf/T_module/T_module.urdf.xacro" />
+  <!-- I Invert Module -->
+  <xacro:include filename="$(find mr_description)/urdf/I_module/I_invert.urdf.xacro" />
   <!-- T Invert Module -->
   <xacro:include filename="$(find mr_description)/urdf/T_module/T_Invert.urdf.xacro" />
@@ -14,4 +16,6 @@
   <!-- Gripper100 invert Module -->
   <xacro:include filename="$(find mr_description)/urdf/G_invert.urdf.xacro" />
+  <!-- sleeve_link Module -->
+  <xacro:include filename="$(find mr_description)/urdf/sleeve_link.urdf.xacro" />
 <!-- Now we can start using the macros included above to define the actual robot -->
   <!-- The first use of a macro.  This one was defined in base.urdf.xacro above.
@@ -28,20 +32,23 @@
   </xacro:G_invert>
   <xacro:I_module name="_I5" parent="_G6_palm_link">
-    <origin xyz="0 0 0" rpy="${pi*0.5} 0 0" />
+    <origin xyz="0 0 0" rpy="${pi*0.5} ${-pi*0.5} 0" />
   </xacro:I_module>
   <xacro:T_invert name="_T4" parent="_I5_Lr_Link_3">
     <origin xyz="0 0 0.005" rpy="0 0 0" />
   </xacro:T_invert>
-  <xacro:T_module name="_T3" parent="_T4_Lr_Link_0">
+  <xacro:sleeve_link name="sleeve_link" parent="_T4_Lr_Link_0" >
+    <origin xyz="0 0 0.005" rpy="0 0 0" />
+  </xacro:sleeve_link>
+  <xacro:T_invert name="_T3" parent="sleeve_link_link">
+    <origin xyz="0 0 ${sleeve_link_length+0.005}" rpy="0 0 0" />
+  </xacro:T_invert>
+  <xacro:T_module name="_T2" parent="_T3_Lr_Link_0">
+    <origin xyz="0 0 0.005" rpy="0 0 ${pi}" />
+  </xacro:T_module>
+  <xacro:I_invert name="_I1" parent="_T2_Lr_Link_3">
     <origin xyz="0 0 0" rpy="0 0 0" />
-  </xacro:T_module>
-  <xacro:T_invert name="_T2" parent="_T3_Lr_Link_3">
-    <origin xyz="0 0 0.005" rpy="0 0 0" />
-  </xacro:T_invert>
-  <xacro:I_module name="_I1" parent="_T2_Lr_Link_0">
-    <origin xyz="0 0 0" rpy="0 0 0" />
-  </xacro:I_module>
+  </xacro:I_invert>
   <xacro:G_module name="_G0" parent="_I1_Lr_Link_3">
-    <origin xyz="0 0 0" rpy="${pi*0.5} 0 0" />
+    <origin xyz="0 0 0" rpy="${pi*0.5} 0 ${-pi*0.5}" />
   </xacro:G_module>
 </robot>

File: mr_description/urdf/I_module/I_module.urdf.xacro (robot description, xacro)
@@ -2,5 +2,5 @@
 <robot xmlns:xacro="http://www.ros.org/wiki/xacro">
 <!--definition of default_inertial -->
-<xacro:macro name="I_module" params="parent name *origin">
+<xacro:macro name="I_module" params="parent name *origin rotate_direction_pos:=1">
 <!-- joint between base_link and Lockring_Link -->
 	<joint name="${name}_joint_0" type="fixed" >
@@ -68,5 +68,11 @@
     <parent  link="${name}_InLink_1" />
     <child   link="${name}_OutLink_2" />
-    <axis   xyz="0 0 1" />
+<!--    <xacro:if value="${rotate_direction_pos}">-->
+<!--       <axis   xyz="0 0 1" />-->
+<!--    </xacro:if>-->
+<!--    <xacro:unless value="${rotate_direction_pos}">-->
+<!--       <axis   xyz="0 0 -1" />-->
+<!--    </xacro:unless>-->
+    <axis   xyz="0 0 ${rotate_direction_pos}" />
     <limit   effort="75"  velocity="1.1" />
   </joint>

Commit message: add offset for i_module

File: mr_description/robots/climbot5d.urdf.xacro (robot description, xacro)
@@ -35,5 +35,5 @@
   </xacro:I_module>
   <xacro:T_invert name="T2" parent="I1_Link">
-    <origin xyz="0 0 0.005" rpy="0 0 0" />
+    <origin xyz="0 0 0" rpy="0 0 0" />
   </xacro:T_invert>
   <xacro:T_module name="T3" parent="T2_Link" >

File: mr_description/robots/manipulator5d.urdf.xacro (robot description, xacro)
@@ -39,5 +39,5 @@
   </xacro:I_module>
   <xacro:T_invert name="T2" parent="I1_Link" >
-    <origin xyz="0 0 0" rpy="0 0 0" />
+    <origin xyz="0 0 0.005" rpy="0 0 0" />
   </xacro:T_invert>
   <xacro:T_module name="T3" parent="T2_Link">
@@ -51,5 +51,5 @@
   </xacro:i_module>
   <xacro:t_module name="t5" parent="i4_Link">
-    <origin xyz="0 0 0" rpy="0 0 ${-pi*0.5}" />
+    <origin xyz="0 0 0" rpy="0 0 0" />
   </xacro:t_module>
   <xacro:g_module name="g6" parent="t5_Link">

File: mr_description/urdf/I_module/I_module.urdf.xacro (robot description, xacro)
@@ -112,14 +112,14 @@
 <!--    </collision>-->
   </link>
-<!-- joint between IModule_OutLink and Lockring_Link -->
+<!-- joint between IModule_OutLink and Offset_Link -->
     <joint name="${name}_Lr_Joint_3" type="fixed">
       <origin xyz="0 0 0.0432" rpy="0 0 0" />
       <parent link="${name}_OutLink_2" />
-      <child  link="${name}_Link" />
+      <child  link="${name}_Offset_Link" />
       <axis   xyz="0 0 0" />
       <limit  lower="0" upper="0"  effort="0"   velocity="0" />
     </joint>
-<!--the Lockring_Link in I module-->
-  <link name="${name}_Link">
+<!--the Offset_Link in I module-->
+  <link name="${name}_Offset_Link">
     <inertial>
       <origin  xyz="-1.7347E-18 4.5159E-17 -0.00285"  rpy="0 0 0" />
@@ -142,4 +142,19 @@
 <!--    </collision>-->
   </link>
+<!--Joint between Offset_Link and Lockring_Link-->
+  <joint name="${name}_Offset_Joint" type="fixed">
+    <origin xyz="0 0 0.005" rpy="0 0 0"/>
+    <parent link="${name}_Offset_Link"/>
+    <child link="${name}_Link"/>
+  </joint>
+<!--the Lockring_Link in T module-->
+  <link name="${name}_Link">
+<!--    <collision>-->
+<!--      <origin xyz="0 0 0" rpy="0 0 0" />-->
+<!--      <geometry>-->
+<!--        <mesh filename="package://mr_description/meshes/VT_InLink.STL" />-->
+<!--      </geometry>-->
+<!--    </collision>-->
+  </link>
 </xacro:macro>
 </robot>

File: mr_description/urdf/i_module.urdf.xacro (robot description, xacro)
@@ -1,4 +1,5 @@
 <?xml version="1.0"?>
 <robot xmlns:xacro="http://www.ros.org/wiki/xacro">
+<xacro:property name="pi" value="3.1415926535897931" />
 <!--definition of default_inertial -->
 <xacro:macro name="i_module" params="parent name *origin">
@@ -34,5 +35,5 @@
     </collision>
   </link>
-  <link  name="${name}_Link">
+  <link  name="${name}_Offset_Link">
     <inertial>
       <origin xyz="-2.4633E-14 3.7186E-08 -0.022781" rpy="0 0 0" />
@@ -62,8 +63,23 @@
 <!--    </collision>-->
   </link>
+<!--Joint between Offset_Link and Lockring_Link-->
+  <joint name="${name}_Offset_Joint" type="fixed">
+    <origin xyz="0 0 0" rpy="0 0 ${0.5*pi}"/>
+    <parent link="${name}_Offset_Link"/>
+    <child link="${name}_Link"/>
+  </joint>
+<!--the Lockring_Link in T module-->
+  <link name="${name}_Link">
+<!--    <collision>-->
+<!--      <origin xyz="0 0 0" rpy="0 0 0" />-->
+<!--      <geometry>-->
+<!--        <mesh filename="package://mr_description/meshes/VT_InLink.STL" />-->
+<!--      </geometry>-->
+<!--    </collision>-->
+  </link>
   <joint   name="${name}_Joint"  type="continuous">
     <origin xyz="0 0 0.137" rpy="-8.5591E-29 0 0" />
     <parent  link="${name}_link" />
-    <child   link="${name}_Link" />
+    <child   link="${name}_Offset_Link" />
     <axis    xyz="0 0 1" />
     <limit lower="-3.1416" upper="3.1416" effort="30" velocity="1.29" />

Commit message: add offset for i_module

File: mr_description/robots/climbot5d.urdf.xacro (robot description, xacro)
@@ -38,5 +38,5 @@
   </xacro:T_invert>
   <xacro:T_module name="T3" parent="T2_Link" >
-    <origin xyz="0 0 0.005" rpy="0 0 ${pi}" />
+    <origin xyz="0 0 0" rpy="0 0 ${pi}" />
   </xacro:T_module>
   <xacro:sleeve_link name="sleeve_link" parent="T3_Link" >

File: mr_description/urdf/i_module.urdf.xacro (robot description, xacro)
@@ -65,5 +65,5 @@
 <!--Joint between Offset_Link and Lockring_Link-->
   <joint name="${name}_Offset_Joint" type="fixed">
-    <origin xyz="0 0 0" rpy="0 0 ${0.5*pi}"/>
+    <origin xyz="0 0 0" rpy="0 0 ${-0.5*pi}"/>
     <parent link="${name}_Offset_Link"/>
     <child link="${name}_Link"/>

Commit message: add offset for T_Invert

File: mr_description/robots/climbot5d.urdf.xacro (robot description, xacro)
@@ -38,5 +38,5 @@
   </xacro:T_invert>
   <xacro:T_module name="T3" parent="T2_Link" >
-    <origin xyz="0 0 0" rpy="0 0 ${pi}" />
+    <origin xyz="0 0 0" rpy="0 0 0" />
   </xacro:T_module>
   <xacro:sleeve_link name="sleeve_link" parent="T3_Link" >

File: mr_description/urdf/I_module/I_module.urdf.xacro (robot description, xacro)
@@ -112,14 +112,14 @@
 <!--    </collision>-->
   </link>
-<!-- joint between IModule_OutLink and Offset_Link -->
+<!-- joint between IModule_OutLink and Lockring_Link -->
     <joint name="${name}_Lr_Joint_3" type="fixed">
       <origin xyz="0 0 0.0432" rpy="0 0 0" />
       <parent link="${name}_OutLink_2" />
-      <child  link="${name}_Offset_Link" />
+      <child  link="${name}_Link" />
       <axis   xyz="0 0 0" />
       <limit  lower="0" upper="0"  effort="0"   velocity="0" />
     </joint>
-<!--the Offset_Link in I module-->
-  <link name="${name}_Offset_Link">
+<!--the Lockring_Link in I module-->
+  <link name="${name}_Link">
     <inertial>
       <origin  xyz="-1.7347E-18 4.5159E-17 -0.00285"  rpy="0 0 0" />
@@ -142,19 +142,4 @@
 <!--    </collision>-->
   </link>
-<!--Joint between Offset_Link and Lockring_Link-->
-  <joint name="${name}_Offset_Joint" type="fixed">
-    <origin xyz="0 0 0.005" rpy="0 0 0"/>
-    <parent link="${name}_Offset_Link"/>
-    <child link="${name}_Link"/>
-  </joint>
-<!--the Lockring_Link in T module-->
-  <link name="${name}_Link">
-<!--    <collision>-->
-<!--      <origin xyz="0 0 0" rpy="0 0 0" />-->
-<!--      <geometry>-->
-<!--        <mesh filename="package://mr_description/meshes/VT_InLink.STL" />-->
-<!--      </geometry>-->
-<!--    </collision>-->
-  </link>
 </xacro:macro>
 </robot>

File: mr_description/urdf/T_module/T_Invert.urdf.xacro (robot description, xacro)
@@ -11,6 +11,21 @@
     <child link="${name}_Lr_Link_3" />
   </joint>
+<!--Joint between Offset_Lockring_Link and Lockring_Link-->
+  <joint name="${name}_Offset_Joint2" type="fixed">
+    <origin xyz="0 0 0.005" rpy="0 0 0"/>
+    <parent link="${name}_Lr_Link_3"/>
+    <child link="${name}_Offset_Lr_Link_3"/>
+  </joint>
 <!--the Lockring_Link in T module-->
   <link name="${name}_Lr_Link_3">
+<!--    <collision>-->
+<!--      <origin xyz="0 0 0" rpy="0 0 0" />-->
+<!--      <geometry>-->
+<!--        <mesh filename="package://mr_description/meshes/VT_InLink.STL" />-->
+<!--      </geometry>-->
+<!--    </collision>-->
+  </link>
+<!--the Offset_Lockring_Link in T module-->
+  <link name="${name}_Offset_Lr_Link_3">
     <inertial>
       <origin xyz="-2.7136E-19 9.8046E-20 -0.0015" rpy="0 0 0" />
@@ -37,5 +52,5 @@
       <origin  xyz="0 0 0.0884"  rpy="-${90*pi/180} 3.1416 3.1416" />
       <child link="${name}_OutLink_2" />
-      <parent  link="${name}_Lr_Link_3" />
+      <parent  link="${name}_Offset_Lr_Link_3" />
       <axis   xyz="0 0 0" />
       <limit  lower="0" upper="0"  effort="0"   velocity="0" />
