Commit message: modify module xacro files

File: mr_description/robots/manipulator5d.urdf.xacro (robot description, xacro)
@@ -38,20 +38,20 @@
     <origin xyz="0 0 0" rpy="0 0 0" />
   </xacro:I_module>
-  <xacro:T_invert name="T2" parent="I1_Lr_Link_3" >
+  <xacro:T_invert name="T2" parent="I1_Link" >
     <origin xyz="0 0 0" rpy="0 0 0" />
   </xacro:T_invert>
-  <xacro:T_module name="T3" parent="T2_Lr_Link_0">
+  <xacro:T_module name="T3" parent="T2_Link">
     <origin xyz="0 0 0.005" rpy="0 0 ${pi}" />
   </xacro:T_module>
-  <xacro:connect_link_100_85  name="cl" parent="T3_Lr_Link_3">
+  <xacro:connect_link_100_85  name="cl" parent="T3_Link">
     <origin xyz="0 0 0" rpy="0 0 0" />
   </xacro:connect_link_100_85>
-  <xacro:i_module name="i4" parent="cl_100_85_connect_link2">
+  <xacro:i_module name="i4" parent="cl_100_85_connect_Link">
     <origin xyz="0 0 0" rpy="0 0 0" />
   </xacro:i_module>
-  <xacro:t_module name="t5" parent="i4_link2">
+  <xacro:t_module name="t5" parent="i4_Link">
     <origin xyz="0 0 0" rpy="0 0 ${-pi*0.5}" />
   </xacro:t_module>
-  <xacro:g_module name="g6" parent="t5_link2">
+  <xacro:g_module name="g6" parent="t5_Link">
     <origin xyz="0 0 0.0825" rpy="0 0 0" />
   </xacro:g_module>

File: mr_description/urdf/100_85connect_link.urdf.xacro (robot description, xacro)
@@ -41,11 +41,11 @@
     </collision>
   </link>
-  <link name="${name}_100_85_connect_link2" />
   <joint   name="${name}_fixed" type="fixed">
     <origin xyz="0 0 0.0236" rpy="0 0 0" />
     <parent   link="${name}_100_85_connect_link" />
-    <child    link="${name}_100_85_connect_link2" />
+    <child    link="${name}_100_85_connect_Link" />
     <axis     xyz="0 0 0" />
   </joint>
+  <link name="${name}_100_85_connect_Link" />
   </xacro:macro>
 </robot>

File: mr_description/urdf/I_module/I_module.urdf.xacro (robot description, xacro)
@@ -116,10 +116,10 @@
       <origin xyz="0 0 0.0432" rpy="0 0 0" />
       <parent link="${name}_OutLink_2" />
-      <child  link="${name}_Lr_Link_3" />
+      <child  link="${name}_Link" />
       <axis   xyz="0 0 0" />
       <limit  lower="0" upper="0"  effort="0"   velocity="0" />
     </joint>
 <!--the Lockring_Link in I module-->
-  <link name="${name}_Lr_Link_3">
+  <link name="${name}_Link">
     <inertial>
       <origin  xyz="-1.7347E-18 4.5159E-17 -0.00285"  rpy="0 0 0" />

File: mr_description/urdf/T_module/T_Invert.urdf.xacro (robot description, xacro)
@@ -117,5 +117,5 @@
     <joint name="${name}_Lr_Joint_1" type="fixed">
       <origin xyz="0 0 -0.1416" rpy="0 3.1416 0" />
-      <child link="${name}_Lr_Link_0" />
+      <child link="${name}_Link" />
       <parent  link="${name}_InLink_1" />
       <axis   xyz="0 0 0" />
@@ -123,5 +123,5 @@
     </joint>
   <!--the Lockring_Link in T module-->
-  <link name="${name}_Lr_Link_0">
+  <link name="${name}_Link">
     <inertial>
       <origin xyz="2.9038E-18 -2.1866E-18 0.0015" rpy="0 0 0" />

File: mr_description/urdf/T_module/T_module.urdf.xacro (robot description, xacro)
@@ -116,10 +116,10 @@
       <origin  xyz="0 -0.0934 0"  rpy="-1.5708 0 3.1416" />
       <parent link="${name}_OutLink_2" />
-      <child  link="${name}_Lr_Link_3" />
+      <child  link="${name}_Link" />
       <axis   xyz="0 0 0" />
       <limit  lower="0" upper="0"  effort="0"   velocity="0" />
     </joint>
 <!--the Lockring_Link in T module-->
-  <link name="${name}_Lr_Link_3">
+  <link name="${name}_Link">
     <inertial>
       <origin xyz="-2.7136E-19 9.8046E-20 -0.0015" rpy="0 0 0" />

File: mr_description/urdf/i_module.urdf.xacro (robot description, xacro)
@@ -34,5 +34,5 @@
     </collision>
   </link>
-  <link  name="${name}_link2">
+  <link  name="${name}_Link">
     <inertial>
       <origin xyz="-2.4633E-14 3.7186E-08 -0.022781" rpy="0 0 0" />
@@ -65,5 +65,5 @@
     <origin xyz="0 0 0.137" rpy="-8.5591E-29 0 0" />
     <parent  link="${name}_link" />
-    <child   link="${name}_link2" />
+    <child   link="${name}_Link" />
     <axis    xyz="0 0 1" />
     <limit lower="-3.1416" upper="3.1416" effort="30" velocity="1.29" />

File: mr_description/urdf/t_module.urdf.xacro (robot description, xacro)
@@ -33,5 +33,5 @@
     </collision>
   </link>
-  <link name="${name}_link2">
+  <link name="${name}_Link">
     <visual>
       <origin xyz="0 0 0.0825" rpy="0 0 0" />
@@ -60,5 +60,5 @@
     <origin xyz="0 0 0.131" rpy="0 0 3.1416" />
     <parent link="${name}_link" />
-    <child link="${name}_link2" />
+    <child link="${name}_Link" />
     <axis  xyz="1 0 0" />
     <limit lower="-2.09" upper="2.09" effort="28" velocity="2.09" />

Commit message: add offset for T_Invert and t_module

File: mr_description/robots/manipulator5d.urdf.xacro (robot description, xacro)
@@ -42,5 +42,5 @@
   </xacro:T_invert>
   <xacro:T_module name="T3" parent="T2_Link">
-    <origin xyz="0 0 0.005" rpy="0 0 ${pi}" />
+    <origin xyz="0 0 0" rpy="0 0 ${pi}" />
   </xacro:T_module>
   <xacro:connect_link_100_85  name="cl" parent="T3_Link">
@@ -54,5 +54,5 @@
   </xacro:t_module>
   <xacro:g_module name="g6" parent="t5_Link">
-    <origin xyz="0 0 0.0825" rpy="0 0 0" />
+    <origin xyz="0 0 0" rpy="0 0 0" />
   </xacro:g_module>
   <joint name="tcp_fixed_joint" type="fixed" >

File: mr_description/urdf/T_module/T_Invert.urdf.xacro (robot description, xacro)
@@ -114,14 +114,14 @@
     </collision>
   </link>
-<!-- joint between Lockring_Link and TModule_InLink -->
+<!-- joint between Offset_Link and TModule_InLink -->
     <joint name="${name}_Lr_Joint_1" type="fixed">
       <origin xyz="0 0 -0.1416" rpy="0 3.1416 0" />
-      <child link="${name}_Link" />
+      <child link="${name}_Offset_Link" />
       <parent  link="${name}_InLink_1" />
       <axis   xyz="0 0 0" />
       <limit  lower="0" upper="0"  effort="0"   velocity="0" />
     </joint>
-  <!--the Lockring_Link in T module-->
-  <link name="${name}_Link">
+  <!--the Offset_Link in T module-->
+  <link name="${name}_Offset_Link">
     <inertial>
       <origin xyz="2.9038E-18 -2.1866E-18 0.0015" rpy="0 0 0" />
@@ -144,4 +144,19 @@
 <!--    </collision>-->
   </link>
+<!--Joint between Offset_Link and Lockring_Link-->
+  <joint name="${name}_Offset_Joint" type="fixed">
+    <origin xyz="0 0 0.005" rpy="0 0 0"/>
+    <parent link="${name}_Offset_Link"/>
+    <child link="${name}_Link"/>
+  </joint>
+<!--the Lockring_Link in T module-->
+  <link name="${name}_Link">
+<!--    <collision>-->
+<!--      <origin xyz="0 0 0" rpy="0 0 0" />-->
+<!--      <geometry>-->
+<!--        <mesh filename="package://mr_description/meshes/VT_InLink.STL" />-->
+<!--      </geometry>-->
+<!--    </collision>-->
+  </link>
 </xacro:macro>
 </robot>

File: mr_description/urdf/t_module.urdf.xacro (robot description, xacro)
@@ -33,5 +33,5 @@
     </collision>
   </link>
-  <link name="${name}_Link">
+  <link name="${name}_Offset_Link">
     <visual>
       <origin xyz="0 0 0.0825" rpy="0 0 0" />
@@ -60,5 +60,5 @@
     <origin xyz="0 0 0.131" rpy="0 0 3.1416" />
     <parent link="${name}_link" />
-    <child link="${name}_Link" />
+    <child link="${name}_Offset_Link" />
     <axis  xyz="1 0 0" />
     <limit lower="-2.09" upper="2.09" effort="28" velocity="2.09" />
@@ -80,4 +80,19 @@
     </actuator>
   </transmission>
+<!--Joint between Offset_Link and Lockring_Link-->
+  <joint name="${name}_Offset_Joint" type="fixed">
+    <origin xyz="0 0 0.0825" rpy="0 0 0"/>
+    <parent link="${name}_Offset_Link"/>
+    <child link="${name}_Link"/>
+  </joint>
+<!--the Lockring_Link in T module-->
+  <link name="${name}_Link">
+<!--    <collision>-->
+<!--      <origin xyz="0 0 0" rpy="0 0 0" />-->
+<!--      <geometry>-->
+<!--        <mesh filename="package://mr_description/meshes/VT_InLink.STL" />-->
+<!--      </geometry>-->
+<!--    </collision>-->
+  </link>
   </xacro:macro>
 </robot>

Commit message: add offset for T_Invert

File: mr_description/robots/manipulator5d.urdf.xacro (robot description, xacro)
@@ -39,8 +39,8 @@
   </xacro:I_module>
   <xacro:T_invert name="T2" parent="I1_Link" >
-    <origin xyz="0 0 0.005" rpy="0 0 0" />
+    <origin xyz="0 0 0" rpy="0 0 0" />
   </xacro:T_invert>
   <xacro:T_module name="T3" parent="T2_Link">
-    <origin xyz="0 0 0" rpy="0 0 ${pi}" />
+    <origin xyz="0 0 0" rpy="0 0 0" />
   </xacro:T_module>
   <xacro:connect_link_100_85  name="cl" parent="T3_Link">

File: mr_description/urdf/T_module/T_Invert.urdf.xacro (robot description, xacro)
@@ -146,5 +146,5 @@
 <!--Joint between Offset_Link and Lockring_Link-->
   <joint name="${name}_Offset_Joint" type="fixed">
-    <origin xyz="0 0 0.005" rpy="0 0 0"/>
+    <origin xyz="0 0 0.005" rpy="0 0 ${pi}"/>
     <parent link="${name}_Offset_Link"/>
     <child link="${name}_Link"/>

Commit message: push for sync

File: mr_description/robots/manipulator5d.urdf.xacro (robot description, xacro)
@@ -42,5 +42,5 @@
   </xacro:T_invert>
   <xacro:T_module name="T3" parent="T2_Link">
-    <origin xyz="0 0 0" rpy="0 0 0" />
+    <origin xyz="0 0 0" rpy="0 0 ${pi}" />
   </xacro:T_module>
   <xacro:connect_link_100_85  name="cl" parent="T3_Link">
@@ -48,8 +48,8 @@
   </xacro:connect_link_100_85>
   <xacro:i_module name="i4" parent="cl_100_85_connect_Link">
-    <origin xyz="0 0 0" rpy="0 0 0" />
+    <origin xyz="0 0 0" rpy="0 0 ${pi}" />
   </xacro:i_module>
   <xacro:t_module name="t5" parent="i4_Link">
-    <origin xyz="0 0 0" rpy="0 0 0" />
+    <origin xyz="0 0 0" rpy="0 0 ${pi}" />
   </xacro:t_module>
   <xacro:g_module name="g6" parent="t5_Link">

File: mr_description/urdf/g_module.urdf.xacro (robot description, xacro)
@@ -38,4 +38,24 @@
     </inertial>
   </link>
+  <joint  name="${name}_Joint"  type="prismatic">
+    <origin   xyz="0 0 0"    rpy="0 0 0" />
+    <parent   link="${name}_palm_link" />
+    <child   link="${name}_finger_link" />
+    <axis   xyz="-1 0 0" />
+    <limit    lower="0"  upper="0.06" effort="1" velocity="0.06" />
+<!--    <calibration   rising="1"   falling="1" />-->
+<!--    <dynamics    damping="1"    friction="1" />-->
+<!--    <safety_controller soft_upper="0.06" soft_lower="0" k_position="1" k_velocity="1" />-->
+  </joint>
+  <joint  name="${name}_Joint1"  type="prismatic">
+    <origin   xyz="0 0 0"    rpy="0 0 0" />
+    <parent    link="${name}_palm_link" />
+    <child    link="${name}_finger_link1" />
+    <axis   xyz="1 0 0" />
+    <limit  lower="0"  upper="0.06" effort="1" velocity="0.06" />
+<!--    <calibration  rising="1" />-->
+<!--    <dynamics  damping="1"  friction="1" />-->
+<!--    <safety_controller soft_upper="0.06" soft_lower="0" k_position="1" k_velocity="1" />-->
+  </joint>
   <link  name="${name}_finger_link">
     <visual>
@@ -62,26 +82,5 @@
     </inertial>
   </link>
-  <joint  name="${name}_Joint"  type="prismatic">
-    <origin   xyz="0 0 0"    rpy="0 0 0" />
-    <parent   link="${name}_palm_link" />
-    <child   link="${name}_finger_link" />
-    <axis   xyz="-1 0 0" />
-    <limit    lower="0"  upper="0.06" effort="1" velocity="0.06" />
-<!--    <calibration   rising="1"   falling="1" />-->
-<!--    <dynamics    damping="1"    friction="1" />-->
-<!--    <safety_controller soft_upper="0.06" soft_lower="0" k_position="1" k_velocity="1" />-->
-  </joint>
   <link  name="${name}_finger_link1">
-    <inertial>
-      <origin xyz="0.0142537929479934 3.43816122645394E-05 0.123240994639808" rpy="0 0 0" />
-      <mass  value="0.0587979869361215" />
-      <inertia
-        ixx="4.06348713317454E-05"
-        ixy="4.84294028883443E-09"
-        ixz="-9.16297919179846E-06"
-        iyy="4.29642140065595E-05"
-        iyz="-7.56625401696782E-08"
-        izz="9.72744043633773E-06" />
-    </inertial>
     <visual>
       <origin  xyz="0 0 0"  rpy="0 0 0" />
@@ -99,15 +98,16 @@
       </geometry>
     </collision>
+    <inertial>
+      <origin xyz="0.0142537929479934 3.43816122645394E-05 0.123240994639808" rpy="0 0 0" />
+      <mass  value="0.0587979869361215" />
+      <inertia
+        ixx="4.06348713317454E-05"
+        ixy="4.84294028883443E-09"
+        ixz="-9.16297919179846E-06"
+        iyy="4.29642140065595E-05"
+        iyz="-7.56625401696782E-08"
+        izz="9.72744043633773E-06" />
+    </inertial>
   </link>
-  <joint  name="${name}_Joint1"  type="prismatic">
-    <origin   xyz="0 0 0"    rpy="0 0 0" />
-    <parent    link="${name}_palm_link" />
-    <child    link="${name}_finger_link1" />
-    <axis   xyz="1 0 0" />
-    <limit  lower="0"  upper="0.06" effort="1" velocity="0.06" />
-<!--    <calibration  rising="1" />-->
-<!--    <dynamics  damping="1"  friction="1" />-->
-<!--    <safety_controller soft_upper="0.06" soft_lower="0" k_position="1" k_velocity="1" />-->
-  </joint>
   </xacro:macro>
 </robot>

Commit message: modified manipulator5d.urdf.xacro

File: mr_description/robots/manipulator5d.urdf.xacro (robot description, xacro)
@@ -35,4 +35,10 @@
 <!--    <origin xyz="0 0 0.17836" rpy="${-pi*0.5} 0 0" />-->
 <!--  </xacro:G_invert>-->
+  <joint name="tcp_fixed_joint" type="fixed" >
+    <origin xyz="0 0 0.16" rpy="0 0 0" />
+    <parent link="g6_palm_link" />
+    <child link="tcp" />
+  </joint>
+  <link name="tcp"/>
   <xacro:I_module name="I1" parent="base_link">
     <origin xyz="0 0 0" rpy="0 0 0" />
@@ -56,10 +62,4 @@
     <origin xyz="0 0 0" rpy="0 0 0" />
   </xacro:g_module>
-  <joint name="tcp_fixed_joint" type="fixed" >
-    <origin xyz="0 0 0.16" rpy="0 0 0" />
-    <parent link="g6_palm_link" />
-    <child link="tcp" />
-  </joint>
-  <link name="tcp"/>
 <!--  <xacro:G_module name="G6" parent="T5_Lr_Link_3">-->
 <!--    <origin xyz="0 0 0" rpy="${pi*0.5} 0 ${pi*0.5}" />-->
