Commit message: add round pole detection

File: mr_description/robots/climbot5d_gazebo.urdf.xacro (robot description, xacro)
@@ -18,5 +18,6 @@
   <!-- sleeve_link Module -->
   <xacro:include filename="$(find mr_description)/urdf/sleeve_link.urdf.xacro" />
-<!-- Now we can start using the macros included above to define the actual robot -->
+  <!-- kinect Module -->
+  <xacro:include filename="$(find mr_description)/urdf/kinect.urdf.xacro" />
   <!-- The first use of a macro.  This one was defined in base.urdf.xacro above.
        A macro like this will expand to a set of link and joint definitions, and to additional
@@ -26,48 +27,18 @@
        the origin block defines where the component is w.r.t its parent (in this case the parent
        is the world frame). For more, see http://www.ros.org/wiki/xacro -->
+  <!-- ros_control plugin -->
+  <gazebo>
+    <plugin name="gazebo_ros_control" filename="libgazebo_ros_control.so">
+      <robotNamespace>climbot5d</robotNamespace>
+      <robotSimType>gazebo_ros_control/DefaultRobotHWSim</robotSimType>
+    </plugin>
+  </gazebo>
 <!--    climbot move group 1-->
   <link name="base_gripper1" />
-  <joint  name="pole1_Joint"  type="fixed">
-    <origin  xyz="0 0.18 0" rpy="0 0 0" />
-    <parent link="base_gripper1" />
-    <child  link="pole1" />
-  </joint>
-  <link name="pole1" >
-      <visual>
-      <origin xyz="0 0 0.7" rpy="0 0 ${pi*0.25}" />
-      <geometry>
-	<box size="0.04 0.04 2"/>
-      </geometry>
-      <material name="Blue"/>
-    </visual>
-    <collision>
-      <origin xyz="0 0 0" rpy="0 0 0" />
-      <geometry>
-	<box size="0.04 0.04 2"/>
-      </geometry>
-    </collision>
-  </link>
-  <joint  name="pole2_Joint"  type="fixed">
-    <origin  xyz="0 0.18 0" rpy="0 0 0" />
-    <parent link="base_gripper1" />
-    <child  link="pole2" />
-  </joint>
-  <link name="pole2" >
-      <visual>
-      <origin xyz="0.4 0.1 0.7" rpy="${pi*0.5} ${pi*0.54} ${pi*0.25}" />
-      <geometry>
-	<box size="0.04 0.04 2"/>
-      </geometry>
-      <material name="Blue"/>
-    </visual>
-    <collision>
-      <origin xyz="0 0 0.7" rpy="0 0 ${pi*0.25}" />
-      <geometry>
-	<box size="0.04 0.04 2"/>
-      </geometry>
-    </collision>
-  </link>
+  <xacro:kinect name="kinect1" parent="base_gripper1">
+    <origin xyz="0 -0.01 -0.1" rpy="${pi} 0 ${pi*0.5}" />
+  </xacro:kinect>
   <xacro:G_invert name="G0" parent="base_gripper1">
-    <origin xyz="0 0 0.17836" rpy="0 0 0" />
+    <origin xyz="0 0 0" rpy="0 0 0" />
   </xacro:G_invert>
   <xacro:I_module name="I1" parent="G0_palm_link">
@@ -92,29 +63,6 @@
     <origin xyz="0 0 0" rpy="0 0 0" />
   </xacro:G_module>
-<!--    climbot move group 2-->
-<!--   <link name="base_gripper2" />-->
-<!--   -->
-<!--  <xacro:G_invert name="_G6" parent="base_gripper2">-->
-<!--    <origin xyz="0.2 0 0.17836" rpy="${-pi*0.5} 0 0" />-->
-<!--  </xacro:G_invert>-->
-<!--  <xacro:I_module name="_I5" parent="_G6_palm_link">-->
-<!--    <origin xyz="0 0 0" rpy="${pi*0.5} 0 0" />-->
-<!--  </xacro:I_module>-->
-<!--  <xacro:T_invert name="_T4" parent="_I5_Lr_Link_3">-->
-<!--    <origin xyz="0 0 0.005" rpy="0 0 0" />-->
-<!--  </xacro:T_invert>-->
-<!--  -->
-<!--  <xacro:T_module name="_T3" parent="_T4_Lr_Link_0">-->
-<!--    <origin xyz="0 0 0" rpy="0 0 0" />-->
-<!--  </xacro:T_module>-->
-<!--  <xacro:T_invert name="_T2" parent="_T3_Lr_Link_3">-->
-<!--    <origin xyz="0 0 0.005" rpy="0 0 0" />-->
-<!--  </xacro:T_invert>-->
-<!--  <xacro:I_module name="_I1" parent="_T2_Lr_Link_0">-->
-<!--    <origin xyz="0 0 0" rpy="0 0 0" />-->
-<!--  </xacro:I_module>-->
-<!--  -->
-<!--  <xacro:G_module name="_G0" parent="_I1_Lr_Link_3">-->
-<!--    <origin xyz="0 0 0" rpy="${pi*0.5} 0 0" />-->
-<!--  </xacro:G_module>-->
+  <xacro:kinect name="kinect2" parent="G6_tcp">
+    <origin xyz="0 -0.2 -0.1" rpy="${pi} 0 ${pi*0.5}" />
+  </xacro:kinect>
 </robot>

File: mr_description/urdf/G_invert.urdf.xacro (robot description, xacro)
@@ -45,4 +45,8 @@
     </collision>
   </link>
+  <!--the IModule_InLink Gazebo tag-->
+  <gazebo reference="${name}_palm_link">
+    <material>Gazebo/Black</material>
+  </gazebo>
   <joint name="${name}_offset_joint" type="fixed" >
     <origin xyz="0 0 0" rpy="${pi*0.5} ${-pi*0.5} 0" />
@@ -63,9 +67,10 @@
   </joint>
    <!-- test reduction ratio-->
-  <transmission name="simple_trans">
+  <transmission name="${name}_trans">
     <type>transmission_interface/SimpleTransmission</type>
     <joint name="${name}_Joint">
       <hardwareInterface>PositionJointInterface</hardwareInterface>
       <hardwareInterface>VelocityJointInterface</hardwareInterface>
+      <hardwareInterface>EffortJointInterface</hardwareInterface>
     </joint>
     <actuator name="${name}_motor">
@@ -73,4 +78,5 @@
       <hardwareInterface>PositionJointInterface</hardwareInterface>
       <hardwareInterface>VelocityJointInterface</hardwareInterface>
+      <hardwareInterface>EffortJointInterface</hardwareInterface>
     </actuator>
   </transmission>
@@ -105,4 +111,8 @@
     </collision>
   </link>
+  <!--the IModule_InLink Gazebo tag-->
+  <gazebo reference="${name}_finger_link_l">
+    <material>Gazebo/Black</material>
+  </gazebo>
 <!--  joint between the right finger and the palm-->
   <joint  name="${name}_Joint1" type="prismatic">
@@ -114,4 +124,18 @@
     <dynamics  damping="1" friction="1" />
   </joint>
+  <transmission name="${name}_trans1">
+    <type>transmission_interface/SimpleTransmission</type>
+    <joint name="${name}_Joint1">
+      <hardwareInterface>PositionJointInterface</hardwareInterface>
+      <hardwareInterface>VelocityJointInterface</hardwareInterface>
+      <hardwareInterface>EffortJointInterface</hardwareInterface>
+    </joint>
+    <actuator name="${name}_motor">
+      <mechanicalReduction>400</mechanicalReduction>
+      <hardwareInterface>PositionJointInterface</hardwareInterface>
+      <hardwareInterface>VelocityJointInterface</hardwareInterface>
+      <hardwareInterface>EffortJointInterface</hardwareInterface>
+    </actuator>
+  </transmission>
 <!-- the right finger link-->
   <link name="${name}_finger_link_r">
@@ -145,4 +169,8 @@
     </collision>
   </link>
+  <!--the IModule_InLink Gazebo tag-->
+  <gazebo reference="${name}_finger_link_r">
+    <material>Gazebo/Black</material>
+  </gazebo>
   </xacro:macro>
 </robot>

File: mr_description/urdf/G_module.urdf.xacro (robot description, xacro)
@@ -8,11 +8,11 @@
     <insert_block name="origin" />
     <parent link="${parent}" />
-    <child link="${name}_link" />
+    <child link="${name}_Link" />
   </joint>
-  <link name="${name}_link"/>
+  <link name="${name}_Link"/>
 <!-- joint between parent_link and palm _Link -->
   <joint name="${name}_offset_joint" type="fixed" >
     <origin xyz="0 0 0" rpy="${pi*0.5} 0 ${-pi*0.5}" />
-    <parent link="${name}_link" />
+    <parent link="${name}_Link" />
     <child link="${name}_palm_link" />
   </joint>
@@ -51,4 +51,8 @@
     </collision>
   </link>
+  <!--the IModule_InLink Gazebo tag-->
+  <gazebo reference="${name}_palm_link">
+    <material>Gazebo/Black</material>
+  </gazebo>
 <!--  joint between the palm and the left finger-->
   <joint name="${name}_Joint"  type="prismatic">
@@ -61,9 +65,10 @@
   </joint>
    <!-- test reduction ratio-->
-  <transmission name="simple_trans">
+  <transmission name="${name}_trans">
     <type>transmission_interface/SimpleTransmission</type>
     <joint name="${name}_Joint">
       <hardwareInterface>PositionJointInterface</hardwareInterface>
       <hardwareInterface>VelocityJointInterface</hardwareInterface>
+      <hardwareInterface>EffortJointInterface</hardwareInterface>
     </joint>
     <actuator name="${name}_motor">
@@ -71,4 +76,5 @@
       <hardwareInterface>PositionJointInterface</hardwareInterface>
       <hardwareInterface>VelocityJointInterface</hardwareInterface>
+      <hardwareInterface>EffortJointInterface</hardwareInterface>
     </actuator>
   </transmission>
@@ -104,4 +110,8 @@
     </collision>
   </link>
+  <!--the IModule_InLink Gazebo tag-->
+  <gazebo reference="${name}_finger_link_l">
+    <material>Gazebo/Black</material>
+  </gazebo>
 <!--  joint between the right finger and the palm-->
   <joint  name="${name}_Joint1"  type="prismatic">
@@ -113,4 +123,19 @@
     <dynamics   damping="1" friction="1" />
   </joint>
+   <!-- test reduction ratio-->
+  <transmission name="${name}_trans1">
+    <type>transmission_interface/SimpleTransmission</type>
+    <joint name="${name}_Joint1">
+      <hardwareInterface>PositionJointInterface</hardwareInterface>
+      <hardwareInterface>VelocityJointInterface</hardwareInterface>
+      <hardwareInterface>EffortJointInterface</hardwareInterface>
+    </joint>
+    <actuator name="${name}_motor">
+      <mechanicalReduction>400</mechanicalReduction>
+      <hardwareInterface>PositionJointInterface</hardwareInterface>
+      <hardwareInterface>VelocityJointInterface</hardwareInterface>
+      <hardwareInterface>EffortJointInterface</hardwareInterface>
+    </actuator>
+  </transmission>
 <!-- the right finger link-->
   <link name="${name}_finger_link_r">
@@ -144,4 +169,8 @@
     </collision>
   </link>
+  <!--the IModule_InLink Gazebo tag-->
+  <gazebo reference="${name}_finger_link_r">
+    <material>Gazebo/Black</material>
+  </gazebo>
 <!--    joint between the palm link and the tcp-->
   <joint name="${name}_tcp_joint" type="fixed">

File: mr_description/urdf/I_module/I_invert.urdf.xacro (robot description, xacro)
@@ -56,11 +56,15 @@
     <collision>
 <!--      <origin   xyz="0 0 0"  rpy="0 0 0" />-->
-	<origin   xyz="0 0 0.083"  rpy="0 0 0" />
+	    <origin   xyz="0 0 0.083"  rpy="0 0 0" />
       <geometry>
 <!--        <mesh   filename="package://mr_description/meshes/I_InLink.STL" />-->
-	<cylinder radius="0.05" length="0.158"  />
+	      <cylinder radius="0.05" length="0.158"  />
       </geometry>
     </collision>
   </link>
+  <!--the IModule_InLink Gazebo tag-->
+  <gazebo reference="${name}_InLink_1">
+    <material>Gazebo/Red</material>
+  </gazebo>
 <!-- joint between IModule_InLink and IModule_OutLink -->
   <joint  name="${name}_Joint"  type="continuous">
@@ -75,12 +79,14 @@
 <!--    </xacro:unless>-->
     <axis   xyz="0 0 ${rotate_direction_pos}" />
+    <dynamics damping="0.7"/>
     <limit   effort="75"  velocity="1.1" />
   </joint>
   <!--    test reduction ratio-->
-  <transmission name="simple_trans">
+  <transmission name="${name}_trans">
     <type>transmission_interface/SimpleTransmission</type>
     <joint name="${name}_Joint">
       <hardwareInterface>PositionJointInterface</hardwareInterface>
       <hardwareInterface>VelocityJointInterface</hardwareInterface>
+      <hardwareInterface>EffortJointInterface</hardwareInterface>
     </joint>
     <actuator name="${name}_motor">
@@ -88,4 +94,5 @@
       <hardwareInterface>PositionJointInterface</hardwareInterface>
       <hardwareInterface>VelocityJointInterface</hardwareInterface>
+      <hardwareInterface>EffortJointInterface</hardwareInterface>
     </actuator>
   </transmission>
@@ -112,4 +119,8 @@
 <!--    </collision>-->
   </link>
+ <!--the IModule_InLink Gazebo tag-->
+  <gazebo reference="${name}_OutLink_2">
+    <material>Gazebo/Red</material>
+  </gazebo>
 <!-- joint between IModule_OutLink and Lockring_Link -->
     <joint name="${name}_Lr_Joint_3" type="fixed">

File: mr_description/urdf/I_module/I_module.urdf.xacro (robot description, xacro)
@@ -63,4 +63,8 @@
     </collision>
   </link>
+  <!--the IModule_InLink Gazebo tag-->
+  <gazebo reference="${name}_InLink_1">
+    <material>Gazebo/Red</material>
+  </gazebo>
 <!-- joint between IModule_InLink and IModule_OutLink -->
   <joint  name="${name}_Joint"  type="continuous">
@@ -75,12 +79,14 @@
 <!--    </xacro:unless>-->
     <axis   xyz="0 0 ${rotate_direction_pos}" />
+    <dynamics damping="0.7"/>
     <limit   effort="75"  velocity="1.1" />
   </joint>
   <!--    test reduction ratio-->
-  <transmission name="simple_trans">
+  <transmission name="${name}_trans">
     <type>transmission_interface/SimpleTransmission</type>
     <joint name="${name}_Joint">
       <hardwareInterface>PositionJointInterface</hardwareInterface>
       <hardwareInterface>VelocityJointInterface</hardwareInterface>
+      <hardwareInterface>EffortJointInterface</hardwareInterface>
     </joint>
     <actuator name="${name}_motor">
@@ -88,4 +94,5 @@
       <hardwareInterface>PositionJointInterface</hardwareInterface>
       <hardwareInterface>VelocityJointInterface</hardwareInterface>
+      <hardwareInterface>EffortJointInterface</hardwareInterface>
     </actuator>
   </transmission>
@@ -112,4 +119,8 @@
 <!--    </collision>-->
   </link>
+  <!--the IModule_OutLink Gazebo tag-->
+  <gazebo reference="${name}_OutLink_2">
+    <material>Gazebo/Red</material>
+  </gazebo>
 <!-- joint between IModule_OutLink and Lockring_Link -->
     <joint name="${name}_Lr_Joint_3" type="fixed">

File: mr_description/urdf/T_module/T_invert.urdf.xacro (robot description, xacro)
@@ -80,4 +80,8 @@
     </collision>
   </link>
+    <!--the IModule_InLink Gazebo tag-->
+  <gazebo reference="${name}_OutLink_2">
+    <material>Gazebo/Red</material>
+  </gazebo>
 <!-- joint between TModule_InLink and TModule_OutLink -->
   <joint  name="${name}_Joint"  type="revolute">
@@ -88,4 +92,5 @@
     <axis   xyz="0 -1 0" />
     <limit  lower="-2.07" upper="2.07"  effort="75"  velocity="1.047" />
+    <dynamics damping="0.7"/>
   </joint>
   <!--    test reduction ratio-->
@@ -95,5 +100,5 @@
       <hardwareInterface>PositionJointInterface</hardwareInterface>
       <hardwareInterface>VelocityJointInterface</hardwareInterface>
-<!--      <hardwareInterface>EffortJointInterface</hardwareInterface>-->
+      <hardwareInterface>EffortJointInterface</hardwareInterface>
     </joint>
     <actuator name="${name}_motor">
@@ -101,5 +106,5 @@
       <hardwareInterface>PositionJointInterface</hardwareInterface>
       <hardwareInterface>VelocityJointInterface</hardwareInterface>
-<!--      <hardwareInterface>EffortJointInterface</hardwareInterface>-->
+      <hardwareInterface>EffortJointInterface</hardwareInterface>
     </actuator>
   </transmission>
@@ -129,4 +134,8 @@
     </collision>
   </link>
+  <!--the IModule_InLink Gazebo tag-->
+  <gazebo reference="${name}_InLink_1">
+    <material>Gazebo/Red</material>
+  </gazebo>
 <!-- joint between Offset_Link and TModule_InLink -->
     <joint name="${name}_Lr_Joint_1" type="fixed">

File: mr_description/urdf/T_module/T_module.urdf.xacro (robot description, xacro)
@@ -64,4 +64,8 @@
     </collision>
   </link>
+  <!--the IModule_InLink Gazebo tag-->
+  <gazebo reference="${name}_InLink_1">
+    <material>Gazebo/Red</material>
+  </gazebo>
 <!-- joint between TModule_InLink and TModule_OutLink -->
   <joint  name="${name}_Joint"  type="revolute">
@@ -72,4 +76,5 @@
     <axis   xyz="0 0 -1" />
     <limit  lower="-2.07" upper="2.07"  effort="75"  velocity="1.047" />
+    <dynamics damping="0.7"/>
   </joint>
   <!--    test reduction ratio-->
@@ -79,5 +84,5 @@
       <hardwareInterface>PositionJointInterface</hardwareInterface>
       <hardwareInterface>VelocityJointInterface</hardwareInterface>
-<!--      <hardwareInterface>EffortJointInterface</hardwareInterface>-->
+      <hardwareInterface>EffortJointInterface</hardwareInterface>
     </joint>
     <actuator name="${name}_motor">
@@ -85,5 +90,5 @@
       <hardwareInterface>PositionJointInterface</hardwareInterface>
       <hardwareInterface>VelocityJointInterface</hardwareInterface>
-<!--      <hardwareInterface>EffortJointInterface</hardwareInterface>-->
+      <hardwareInterface>EffortJointInterface</hardwareInterface>
     </actuator>
   </transmission>
@@ -112,4 +117,8 @@
     </collision>
   </link>
+  <!--the IModule_InLink Gazebo tag-->
+  <gazebo reference="${name}_OutLink_2">
+    <material>Gazebo/Red</material>
+  </gazebo>
 <!-- joint between TModule_OutLink and Lockring_Link -->
     <joint name="${name}_Lr_Joint_3" type="fixed">

File: mr_description/urdf/i_module.urdf.xacro (robot description, xacro)
@@ -89,9 +89,10 @@
   </joint>
     <!--    test reduction ratio-->
-  <transmission name="simple_trans">
+  <transmission name="${name}_trans">
     <type>transmission_interface/SimpleTransmission</type>
     <joint name="${name}_Joint">
       <hardwareInterface>PositionJointInterface</hardwareInterface>
       <hardwareInterface>VelocityJointInterface</hardwareInterface>
+      <hardwareInterface>EffortJointInterface</hardwareInterface>
     </joint>
     <actuator name="${name}_motor">
@@ -99,4 +100,5 @@
       <hardwareInterface>PositionJointInterface</hardwareInterface>
       <hardwareInterface>VelocityJointInterface</hardwareInterface>
+      <hardwareInterface>EffortJointInterface</hardwareInterface>
     </actuator>
   </transmission>

File: mr_description/urdf/sleeve_link.urdf.xacro (robot description, xacro)
@@ -26,4 +26,8 @@
     </collision>
   </link>
+  <!--the IModule_InLink Gazebo tag-->
+  <gazebo reference="${name}_link">
+    <material>Gazebo/Red</material>
+  </gazebo>
 <!-- offset joint -->
   <joint name="${name}_offset_joint" type="fixed" >

File: mr_description/urdf/t_module.urdf.xacro (robot description, xacro)
@@ -68,9 +68,10 @@
   </joint>
   <!--  reduction ratio-->
-  <transmission name="simple_trans">
+  <transmission name="${name}_trans">
     <type>transmission_interface/SimpleTransmission</type>
     <joint name="${name}_Joint">
       <hardwareInterface>PositionJointInterface</hardwareInterface>
       <hardwareInterface>VelocityJointInterface</hardwareInterface>
+      <hardwareInterface>EffortJointInterface</hardwareInterface>
     </joint>
     <actuator name="${name}_motor">
@@ -78,4 +79,5 @@
       <hardwareInterface>PositionJointInterface</hardwareInterface>
       <hardwareInterface>VelocityJointInterface</hardwareInterface>
+      <hardwareInterface>EffortJointInterface</hardwareInterface>
     </actuator>
   </transmission>
